File: circuit/dap_link.sch (KiCad schematic (older format))
At the start: 35 parts, among them J1 USB_A_CONN, J2 SWD_CONN_5P, J3 UART1_CONN_3P, J4 PAEX_CONN_8P, U1 STM32F103CBTx, U2 AMS1117-3.3, Y1 8MHz

Commit message: ready to print
Parts:
- Y1: footprint Crystal:Crystal_SMD_SeikoEpson_MC405-2Pin_9.6x4.1mm -> Crystal:Crystal_SMD_HC49-SD
Changed lines of the file:
@@
 F 0 "Y1" V 1854 2981 50  0000 L CNN
 F 1 "8MHz" V 1945 2981 50  0000 L CNN
-F 2 "Crystal:Crystal_SMD_SeikoEpson_MC405-2Pin_9.6x4.1mm" H 1900 2850 50  0001 C CNN
+F 2 "Crystal:Crystal_SMD_HC49-SD" H 1900 2850 50  0001 C CNN
 F 3 "~" H 1900 2850 50  0001 C CNN
 	1    1900 2850
