File: circuit/dap_link.kicad_pcb (KiCad board)
At the start: 2 copper layers, 27 parts, among them J1 USB_A_CONN, J2 SWD_CONN_5P, J3 UART1_CONN_3P, U1 STM32F103CBTx, U2 AMS1117-3.3, Y1 8MHz

Commit message: 1
Parts:
- added J4: PAEX_CONN_6P, Connector_PinHeader_2.54mm:PinHeader_1x06_P2.54mm_Vertical, F.Cu at (137.7, 127.5)
- added R11: 1K, Resistor_SMD:R_0603_1608Metric_Pad1.05x0.95mm_HandSolder, F.Cu at (137.7, 121.8)
- added R13: 1K, Resistor_SMD:R_0603_1608Metric_Pad1.05x0.95mm_HandSolder, F.Cu at (140.2, 121.8)
- added R14: 1K, Resistor_SMD:R_0603_1608Metric_Pad1.05x0.95mm_HandSolder, F.Cu at (142.7, 121.8)
- added R15: 1K, Resistor_SMD:R_0603_1608Metric_Pad1.05x0.95mm_HandSolder, F.Cu at (145.3, 121.8)
- added R16: 1K, Resistor_SMD:R_0603_1608Metric_Pad1.05x0.95mm_HandSolder, F.Cu at (147.8, 121.8)
- moved J1 68.2 mm to (185.4, 104.1)
- moved U2 44.6 mm to (163.8, 121.9), turned to 270 degrees
- moved C6 41.4 mm to (157.1, 114.3), turned to 90 degrees
- moved U1 19.6 mm to (146.1, 111.8)
- moved J2 9.02 mm to (140.5, 75.9), turned to 90 degrees
Connections:
- U1 pad 10: Net-(U1-Pad10) -> /PA0
- U1 pad 11: Net-(U1-Pad11) -> /PA1
- U1 pad 12: Net-(U1-Pad12) -> /PA2
- U1 pad 13: Net-(U1-Pad13) -> /PA3
- U1 pad 14: Net-(U1-Pad14) -> /PA4

Commit message: DA111
Parts:
- added R17: 1K, Resistor_SMD:R_0603_1608Metric_Pad1.05x0.95mm_HandSolder, F.Cu at (175.7, 66.8)
- added R18: 1K, Resistor_SMD:R_0603_1608Metric_Pad1.05x0.95mm_HandSolder, F.Cu at (175.7, 69.3)
- J4: value PAEX_CONN_6P -> PAEX_CONN_8P; footprint Connector_PinHeader_2.54mm:PinHeader_1x06_P2.54mm_Vertical -> Connector_PinHeader_2.54mm:PinHeader_1x08_P2.54mm_Vertical
Connections:
- J4 pad 6: GND -> Net-(J4-Pad6)
- U1 pad 15: Net-(U1-Pad15) -> /PA5
- U1 pad 16: /LEDR_GPIO -> /PA6
- U1 pad 17: /LEDG_GPIO -> /LEDR_GPIO
- U1 pad 29: Net-(U1-Pad29) -> /LEDG_GPIO

Commit message: 1
Parts:
- J4: footprint Connector_PinHeader_2.54mm:PinHeader_1x08_P2.54mm_Vertical -> Connector_PinHeader_2.54mm:PinHeader_1x08_P2.54mm_Horizontal
- Y1: footprint Crystal:Crystal_SMD_SeikoEpson_MA505-2Pin_12.7x5.1mm -> Crystal:Crystal_SMD_SeikoEpson_MC405-2Pin_9.6x4.1mm
- moved J1 100.4 mm to (87.8, 127.5), turned to 180 degrees
- moved R17 68.8 mm to (131.0, 119.1)
- moved R18 65.6 mm to (131.0, 117.4)
- moved J2 63.2 mm to (123.2, 136.7)
- moved J3 62.4 mm to (118.4, 136.7), turned to 270 degrees
- moved U2 59.9 mm to (105.3, 134.8), turned to 180 degrees
- moved R7 56.7 mm to (120.7, 132.6), turned to 90 degrees
- moved R4 54.8 mm to (101.6, 123.8), turned to 270 degrees
- moved R8 52.0 mm to (108.2, 119.5)
- moved C7 51.4 mm to (126.0, 127.3), turned to 180 degrees
- moved C1 51.3 mm to (96.8, 117.5)
- moved C3 51.1 mm to (122.6, 122.1), turned to 90 degrees
- moved R1 48.4 mm to (96.8, 119.2)
- moved D2 47.6 mm to (104.3, 117.5), turned to 180 degrees
- moved R2 47.6 mm to (102.6, 128.6), turned to 180 degrees
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Connections:
- net Net-(J1-Pad2) renamed /USB_CONN_D-
- net Net-(J1-Pad3) renamed /USB_CONN_D+
- C5 pad 1: Net-(C5-Pad1) -> +5V
- J1 pad 1: Net-(J1-Pad1) -> +5V
- J2 pad 1: +3V3 -> GND
- J2 pad 2: /NRST -> /SWCLK
- J2 pad 4: /SWCLK -> /NRST
- J2 pad 5: GND -> +3V3
- J3 pad 1: /UTX1 -> GND
- J3 pad 3: GND -> /UTX1
- J4 pad 1: Net-(J4-Pad1) -> GND
- J4 pad 8: GND -> Net-(J4-Pad8)
- R11 pad 2: Net-(J4-Pad1) -> Net-(J4-Pad8)
- R13 pad 2: Net-(J4-Pad2) -> Net-(J4-Pad7)
- R14 pad 2: Net-(J4-Pad3) -> Net-(J4-Pad6)
- R15 pad 2: Net-(J4-Pad4) -> Net-(J4-Pad5)
- R16 pad 2: Net-(J4-Pad5) -> Net-(J4-Pad4)
- R17 pad 2: Net-(J4-Pad6) -> Net-(J4-Pad3)
- R18 pad 2: Net-(J4-Pad7) -> Net-(J4-Pad2)
- U2 pad 3: Net-(C5-Pad1) -> +5V
Other:
- board outline added: 60 x 23.5 mm
- rule solder_mask_min_width: 0.25 -> 0.1

Commit message: 1333
Parts:
- C1, C4, C5, C6, C7, J1, R1, R5, U2, Y1: moved to B.Cu
- moved R1 18.5 mm to (97.4, 137.7)
- moved C1 18.5 mm to (97.4, 135.9)
- moved C5 18.2 mm to (100.2, 118.7), turned to 0 degrees
- moved R6 17.9 mm to (100.8, 134.2), turned to 0 degrees
- moved J4 15.7 mm to (134.5, 118.7)
- moved R7 14.4 mm to (106.3, 134.2), turned to 0 degrees
- moved U2 14.4 mm to (109.0, 120.8)
- moved C8 12.8 mm to (122.6, 131.8), turned to 90 degrees
- moved R10 12.7 mm to (120.9, 131.8), turned to 270 degrees
- moved C6 12.6 mm to (117.6, 120.8)
- moved J3 11.5 mm to (106.9, 136.9)
- moved R12 11.1 mm to (112.5, 137.1), turned to 180 degrees
- moved Y1 8.47 mm to (123.3, 126.9), turned to 90 degrees
- moved R4 7.54 mm to (102.4, 131.3), turned to 90 degrees
- moved C2 7.47 mm to (121.8, 129.1), turned to 180 degrees
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Connections:
- net /USB_CONN_D+ renamed Net-(J1-Pad3)
- net /USB_CONN_D- renamed Net-(J1-Pad2)
Routing:
- net +3V3: track 0.00 -> 76.0 mm, vias 0 -> 3
- net /SWDIO: track 0.00 -> 21.5 mm, vias 0 -> 2
- net +5V: track 0.00 -> 20.9 mm
- net /PA6: track 0.00 -> 15.7 mm
- net /NRST: track 0.00 -> 15.1 mm
- net /PA5: track 0.00 -> 14.5 mm
- net Net-(R7-Pad2): track 0.00 -> 13.6 mm, vias 0 -> 2
- net /PA4: track 0.00 -> 13.2 mm
- net /OSC_IN: track 0.00 -> 12.8 mm, vias 0 -> 1
- net /SWCLK: track 0.00 -> 12.3 mm, vias 0 -> 2
- net Net-(C7-Pad1): track 0.00 -> 11.9 mm
- net /PA3: track 0.00 -> 11.6 mm
- net Net-(R6-Pad2): track 0.00 -> 11.6 mm, vias 0 -> 2
- net /PA0: track 0.00 -> 11.1 mm
- net /LEDG_GPIO: track 0.00 -> 10.9 mm
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- added copper zone on B.Cu, net GND
- added copper zone on F.Cu, net GND
Other:
- board size 60 x 23.5 mm -> 47.3 x 23.5 mm

Commit message: pcb almost done
Parts:
- moved R11 0.10 mm to (127.8, 128.9)
Routing:
- net Net-(C1-Pad1): track 5.38 -> 19.3 mm
- net GND: track 4.23 -> 12.9 mm, vias 2 -> 3
- net /SWDIO: track 21.5 -> 17.3 mm
- net Net-(R7-Pad2): track 13.6 -> 11.0 mm
- net +3V3: track 76.0 -> 77.9 mm

Commit message: ready to print
Parts:
- Y1: footprint Crystal:Crystal_SMD_SeikoEpson_MC405-2Pin_9.6x4.1mm -> Crystal:Crystal_SMD_HC49-SD
- moved Y1 0.98 mm to (123.9, 126.1)
Routing:
- net Net-(C7-Pad1): track 11.9 -> 13.5 mm
Other:
- board size 47.3 x 23.5 mm -> 44.6 x 23.5 mm
