File: circuit/dap_link.kicad_pcb (KiCad board)
At the start: 2 copper layers, 44.6 x 23.5 mm, 35 parts, among them J1 USB_A_CONN, J2 SWD_CONN_5P, J3 UART1_CONN_3P, J4 PAEX_CONN_8P, U1 STM32F103CBTx, U2 AMS1117-3.3, Y1 8MHz

Commit message: pcb done
Routing:
- net +3V3: track 77.9 -> 75.7 mm
Other:
- board text added: "3.3V"
- board text added: "CLK"
- board text added: "DIO"
- board text added: "RST"
- board text added: "RX1"
- board text added: "TX1"
